Commit message: add inertial :books:

File: description/robot.urdf.xacro (robot description, xacro)
@@ -1,4 +1,7 @@
 <?xml version="1.0"?>
 <robot xmlns:xacro="http://www.ros.org/wiki/xacro"  name="robot">
+    <!-- corpo do robo (principal)-->
     <xacro:include filename="robot_core.xacro" />
+    <!-- inercia do robo -->
+    <xacro:include filename="inertial_macros.xacro" />
 </robot>

File: description/robot_core.xacro (robot description, xacro)
@@ -39,4 +39,8 @@
             </geometry>
         </collision>
+        <!-- adicionando a inercia ao robo-->
+        <xacro:inertial_box mass="0.5" x="0.3" y="0.3" z="0.15">
+            <origin xyz="0.15 0 0.075" rpy="0 0 0"/>
+        </xacro:inertial_box>
     </link>
     <!-- === RODA ESQUERDA  === -->
@@ -60,4 +64,7 @@
             <material name="blue"/>
         </collision>
+        <xacro:inertial_cylinder mass="0.1" length="0.05" radius="0.05">
+            <origin xyz="0 0 0" rpy="0 0 0"/>
+        </xacro:inertial_cylinder>
     </link>
     <!-- === RODA DIREITA  === -->
@@ -81,4 +88,7 @@
             <material name="blue"/>
         </collision>
+        <xacro:inertial_cylinder mass="0.1" length="0.05" radius="0.05">
+            <origin xyz="0 0 0" rpy="0 0 0"/>
+        </xacro:inertial_cylinder>
     </link>
     <!-- === RODA RODIZIO (roda que conduz o robo) ===  -->
@@ -101,4 +111,7 @@
             <material name="black"/>
         </collision>
+        <xacro:inertial_sphere mass="0.1" radius="0.05">
+            <origin xyz="0 0 0" rpy="0 0 0"/>
+        </xacro:inertial_sphere>
     </link>
 </robot>

Commit message: conect Gazebo

File: description/robot.urdf.xacro (robot description, xacro)
@@ -1,7 +1,7 @@
 <?xml version="1.0"?>
 <robot xmlns:xacro="http://www.ros.org/wiki/xacro"  name="robot">
+    <!-- inercia do robo -->
+    <xacro:include filename="inertial_macros.xacro" />
     <!-- corpo do robo (principal)-->
     <xacro:include filename="robot_core.xacro" />
-    <!-- inercia do robo -->
-    <xacro:include filename="inertial_macros.xacro" />
 </robot>

File: description/robot_core.xacro (robot description, xacro)
@@ -44,4 +44,7 @@
         </xacro:inertial_box>
     </link>
+    <gazebo reference="chassis">
+        <material>Gazebo/White</material>
+    </gazebo>
     <!-- === RODA ESQUERDA  === -->
     <joint name="left_wheel_joint" type="continuous">
@@ -68,4 +71,7 @@
         </xacro:inertial_cylinder>
     </link>
+    <gazebo reference="left_wheel">
+        <material>Gazebo/Yellow</material>
+    </gazebo>
     <!-- === RODA DIREITA  === -->
     <joint name="right_wheel_joint" type="continuous"> <!-- continuous pois a roda se move -->
@@ -92,4 +98,7 @@
         </xacro:inertial_cylinder>
     </link>
+    <gazebo reference="right_wheel">
+        <material>Gazebo/Yellow</material>
+    </gazebo>
     <!-- === RODA RODIZIO (roda que conduz o robo) ===  -->
     <joint name="caster_wheel_joint" type="fixed">
@@ -115,3 +124,8 @@
         </xacro:inertial_sphere>
     </link>
+    <gazebo reference="caster_wheel">
+        <material>Gazebo/Blue</material>
+        <mu1 value="0.001"/> <!-- Atrito da esfero da roda de rodizio-->
+        <mu2 value="0.001"/>
+    </gazebo>
 </robot>

Commit message: add sensor scan :mag_right:

File: description/robot.urdf.xacro (robot description, xacro)
@@ -1,10 +1,9 @@
 <?xml version="1.0"?>
 <robot xmlns:xacro="http://www.ros.org/wiki/xacro"  name="robot">
-    <!-- inercia do robo -->
-    <xacro:include filename="inertial_macros.xacro" />
     <!-- corpo do robo (principal)-->
     <xacro:include filename="robot_core.xacro" />
-    <!-- adicionando controle do robo
+    <!-- adicionando controle do robo -->
     <xacro:include filename="gazebo_control.xacro" />
-    -->
+    <!-- adicionando o sensor lidar -->
+    <xacro:include filename="lidar.xacro" />
 </robot>

File: description/robot_core.xacro (robot description, xacro)
@@ -1,4 +1,6 @@
 <?xml version="1.0"?>
 <robot xmlns:xacro="http://www.ros.org/wiki/xacro">
+    <!-- inercia do robo -->
+    <xacro:include filename="inertial_macros.xacro"/>
    <!-- ============  Cores ==============-->
     <material name="white">
@@ -13,4 +15,7 @@
     <material name="black">
         <color rgba="0 0 0 1"/>
+    </material>
+    <material name="red">
+        <color rgba="1 0 0 1"/>
     </material>
     <!-- ============== BASE DO ROBO ============== -->

Commit message: refresh ros2_control :wrench:

File: description/robot.urdf.xacro (robot description, xacro)
@@ -1,6 +1,4 @@
 <?xml version="1.0"?>
 <robot xmlns:xacro="http://www.ros.org/wiki/xacro"  name="robot">
-    <!-- adicionando camera ao robo -->
-    <xacro:include filename="camera.xacro" />
     <!-- corpo do robo (principal)-->
     <xacro:include filename="robot_core.xacro" />
@@ -8,6 +6,9 @@
     <xacro:include filename="ros2_control.xacro" />
     <!-- adicionando controle do robo
-    <xacro:include filename="gazebo_control.xacro" />   -->
+    <xacro:include filename="gazebo_control.xacro" />
+    -->
     <!-- adicionando o sensor lidar -->
     <xacro:include filename="lidar.xacro" />
+    <!-- adicionando camera ao robo -->
+    <xacro:include filename="camera.xacro" />
 </robot>

File: description/ros2_control.xacro (robot description, xacro)
@@ -5,25 +5,27 @@
             <plugin>gazebo_ros2_control/GazeboSystem</plugin>
         </hardware>
-    </ros2_control>
-    <joint name="left_wheel_joint">
-        <command_interface name="velocity">
-            <param name="min">-10</param>
-            <param name="max">10</param>
-        </command_interface>
-        <state_interface name="position" />
-        <state_interface name="velocity" />
-    </joint>
-    <joint name="right_wheel_joint">
-        <command_interface name="velocity">
-            <param name="min">-10</param>
-            <param name="max">10</param>
-        </command_interface>
-        <state_interface name="velocity" />
-        <state_interface name="position" />
-    </joint>
-    <gazebo>
-        <plugin filename="libgazebo_ros2_control.so" name="gazebo_ros2_control">
-            <parameters>...to be filled in soon!...</parameters>
-        </plugin>
-    </gazebo>
+        <joint name="left_wheel_joint">
+            <command_interface name="velocity">
+                <param name="min">-10</param>
+                <param name="max">10</param>
+            </command_interface>
+            <state_interface name="position" />
+            <state_interface name="velocity" />
+        </joint>
+        <joint name="right_wheel_joint">
+            <command_interface name="velocity">
+                <param name="min">-10</param>
+                <param name="max">10</param>
+            </command_interface>
+            <state_interface name="velocity" />
+            <state_interface name="position" />
+        </joint>
+        <!--
+        <gazebo>
+            <plugin filename="libgazebo_ros2_control.so" name="gazebo_ros2_control">
+                <parameters>$(find articubot_one)/config/my_controllers.yaml</parameters>
+            </plugin>
+        </gazebo>
+        </ros2_control>
+    -->
 </robot>
